File: Ozma.kicad_pcb (KiCad board)
At the start: 2 copper layers, 165.9 x 122.9 mm, 142 parts, among them J1 MJ-4PP-9-Lily58-cache, P1 OLED, P2 OLED, P3 OLED, SW1 SW_Push, SW2 Rotary_Encoder_Switch, U1 W25Q128JVS, U2 RP2040, U3 NCP1117-3.3_SOT223, U4 USBLC6-2SC6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

Commit message: Trace Work Started
Parts:
- turned D21 to 0 degrees
- turned D22 to 0 degrees
- turned D23 to 0 degrees
- turned D36 to 0 degrees
- turned D38 to 0 degrees
- turned D51 to 0 degrees
- turned D53 to 0 degrees
- turned D56 to 0 degrees
- turned D58 to 0 degrees
- turned D6 to 0 degrees
- turned D63 to 0 degrees
- turned D69 to 135 degrees
- turned D7 to 0 degrees
- turned D8 to 0 degrees
- turned D9 to 0 degrees
Connections:
- D48 pad 2: Net-(D48-Pad2) -> Net-(SW2-PadS2)
- MX35 pad 2: Net-(D48-Pad2) -> Net-(SW2-PadS2)
- SW2 pad S1: Net-(D48-Pad2) -> COL6
- SW2 pad S2: COL6 -> Net-(SW2-PadS2)
Routing:
- net ROW3: track 0.00 -> 139.8 mm, vias 0 -> 6
- net ROW2: track 0.00 -> 139.3 mm, vias 0 -> 6
- net ROW4: track 0.00 -> 135.9 mm, vias 0 -> 6
- net ROW1: track 0.00 -> 134.9 mm, vias 0 -> 6
- net ROW0: track 0.00 -> 131.9 mm
- net COL1: track 0.00 -> 114.2 mm, vias 0 -> 5
- net COL6: track 0.00 -> 113.8 mm, vias 0 -> 2
- net COL2: track 0.00 -> 112.1 mm, vias 0 -> 5
- net COL0: track 0.00 -> 106.2 mm, vias 0 -> 5
- net COL4: track 0.00 -> 100.3 mm, vias 0 -> 4
- net COL3: track 0.00 -> 98.4 mm, vias 0 -> 4
- net COL5: track 0.00 -> 97.7 mm, vias 0 -> 4
- net Net-(D47-Pad2): track 0.00 -> 78.1 mm, vias 0 -> 3
- net Net-(D45-Pad2): track 0.00 -> 48.6 mm, vias 0 -> 2
- net Net-(D46-Pad2): track 0.00 -> 47.4 mm, vias 0 -> 3
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