File: Ozma.kicad_sch (KiCad schematic)
At the start: 142 parts, among them J1 MJ-4PP-9-Lily58-cache, P1 OLED, P2 OLED, P3 OLED, SW1 SW_Push, SW2 Rotary_Encoder_Switch, U1 W25Q128JVS, U2 RP2040, U3 NCP1117-3.3_SOT223, U4 USBLC6-2SC6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

Commit message: Trace Work Started
Connections:
- net COL6: now also SW2.S1; no longer SW2.S2
- net at D48.2 (A), MX35.2 (ROW): now also SW2.S2; no longer SW2.S1
Changed lines of the file:
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@@
-(kicad_sch (version 20210621) (generator eeschema)
+(kicad_sch (version 20210615) (generator eeschema)
   (paper "A3")
   (junction (at 24.13 110.49) (diameter 0.9144) (color 0 0 0 0))
@@
     (stroke (width 0) (type solid) (color 0 0 0 0))
   )
-  (wire (pts (xy 323.85 72.39) (xy 340.36 72.39))
-    (stroke (width 0) (type solid) (color 0 0 0 0))
-  )
   (wire (pts (xy 323.85 76.2) (xy 316.23 76.2))
     (stroke (width 0) (type solid) (color 0 0 0 0))
@@
     (stroke (width 0) (type solid) (color 0 0 0 0))
   )
+  (wire (pts (xy 325.12 69.85) (xy 325.12 72.39))
+    (stroke (width 0) (type solid) (color 0 0 0 0))
+  )
+  (wire (pts (xy 325.12 72.39) (xy 323.85 72.39))
+    (stroke (width 0) (type solid) (color 0 0 0 0))
+  )
   (wire (pts (xy 326.39 25.4) (xy 326.39 33.02))
     (stroke (width 0) (type solid) (color 0 0 0 0))
@@
     (stroke (width 0) (type solid) (color 0 0 0 0))
   )
+  (wire (pts (xy 330.2 67.31) (xy 326.39 67.31))
+    (stroke (width 0) (type solid) (color 0 0 0 0))
+  )
+  (wire (pts (xy 330.2 72.39) (xy 330.2 67.31))
+    (stroke (width 0) (type solid) (color 0 0 0 0))
+  )
+  (wire (pts (xy 330.2 72.39) (xy 340.36 72.39))
+    (stroke (width 0) (type solid) (color 0 0 0 0))
+  )
+  (wire (pts (xy 336.55 67.31) (xy 336.55 69.85))
+    (stroke (width 0) (type solid) (color 0 0 0 0))
+  )
+  (wire (pts (xy 336.55 69.85) (xy 325.12 69.85))
+    (stroke (width 0) (type solid) (color 0 0 0 0))
+  )
   (wire (pts (xy 339.09 90.17) (xy 354.33 90.17))
     (stroke (width 0) (type solid) (color 0 0 0 0))
@@
     (stroke (width 0) (type solid) (color 0 0 0 0))
   )
-  (wire (pts (xy 340.36 67.31) (xy 326.39 67.31))
-    (stroke (width 0) (type solid) (color 0 0 0 0))
-  )
+  (wire (pts (xy 340.36 67.31) (xy 336.55 67.31))
+    (stroke (width 0) (type solid) (color 0 0 0 0))
+  )
